Commit message: joints need offset, not wheels

File: src/chap4_rviz_basics/urdf/gpgMin.urdf (robot description, URDF)
Before this commit: robot gpgMin, 3 links, 2 joints
Joints:
- joint joint_left_wheel: origin xyz=0 0 0 rpy=0 0 0 -> xyz=0.020 0.058 -0.035 rpy=0 0 0
- joint joint_right_wheel: origin xyz=0 0 0 rpy=0 0 0 -> xyz=0.020 -0.058 -0.035 rpy=0 0 0
