Commit message: added laser_frame and levels 2 and 3

File: src/chap4_rviz_basics/urdf/dave.urdf (robot description, URDF)
Before this commit: robot dave, 4 links, 3 joints
Links:
- added link laser_frame; visual cylinder length=0.020 radius=0.0325
- link base_link: geometry visual box size=0.020 0.040 0.025; visual box size=0.025 0.055 0.026
Joints:
- added joint joint_ydlidar: type fixed, parent base_link, child laser_frame, origin xyz=0 0 0.200 rpy=0 0 0
- joint joint_distance_sensor: origin xyz=0.095 0.0 0.100 rpy=0 0 0 -> xyz=0.11 0.0 0.140 rpy=0 0 0
- joint joint_left_wheel: origin xyz=0.020 0.058 -0.035 rpy=0 0 0 -> xyz=0.020 0.058 0.0325 rpy=0 0 0
- joint joint_right_wheel: origin xyz=0.020 -0.058 -0.035 rpy=0 0 0 -> xyz=0.020 -0.058 0.0325 rpy=0 0 0

Commit message: wheels as 0

File: src/chap4_rviz_basics/urdf/dave.urdf (robot description, URDF)
Before this commit: robot dave, 5 links, 4 joints
Links:
- link base_link: geometry visual box size=0.020 0.040 0.025; visual box size=0.025 0.055 0.002
- link left_wheel: geometry visual cylinder length=0.025 radius=0.03385
- link right_wheel: geometry visual cylinder length=0.025 radius=0.033385
Joints:
- joint joint_distance_sensor: origin xyz=0.11 0.0 0.140 rpy=0 0 0 -> xyz=0.081 0.0 0.140 rpy=0 0 0
- joint joint_left_wheel: origin xyz=0.020 0.058 0.0325 rpy=0 0 0 -> xyz=0 0.058 0.033385 rpy=0 0 0
- joint joint_right_wheel: origin xyz=0.020 -0.058 0.0325 rpy=0 0 0 -> xyz=0 -0.058 0.033385 rpy=0 0 0
- joint joint_ydlidar: origin xyz=0 0 0.200 rpy=0 0 0 -> xyz=-0.014 0 0.200 rpy=0 0 0

Commit message: dist sensor seems good now

File: src/chap4_rviz_basics/urdf/dave.urdf (robot description, URDF)
Before this commit: robot dave, 5 links, 4 joints
Joints:
- joint joint_distance_sensor: origin xyz=0.081 0.0 0.140 rpy=0 0 0 -> xyz=0.080 0.0 0.125 rpy=0 0 0

Commit message: added ultrasound

File: src/chap4_rviz_basics/urdf/dave.urdf (robot description, URDF)
Before this commit: robot dave, 5 links, 4 joints
Links:
- added link ultrasonic_ranger; visual box size=0.002 0.035 0.023
Joints:
- added joint joint_ultrasonic: type fixed, parent base_link, child ultrasonic_ranger, origin xyz=-0.080 0 0.125 rpy=0 0 0

Commit message: added imu to urdf

File: src/chap4_rviz_basics/urdf/dave.urdf (robot description, URDF)
Before this commit: robot dave, 6 links, 5 joints
Links:
- added link imu_link; visual box size=0.023 0.035 0.002
Joints:
- added joint joint_imu: type fixed, parent base_link, child imu_link, origin xyz=0.070 0.035 0.055 rpy=0 0 0
- joint joint_ultrasonic: origin xyz=-0.080 0 0.125 rpy=0 0 0 -> xyz=0.093 0 0.110 rpy=0 0 0
